File: hw/ecu/ecu.kicad_pcb (KiCad board)
At the start: 2 copper layers, 143.8 x 80 mm, 269 parts, among them J1 POWER, J10 CUR_LOOP_IN, J11 SENSORS, J12 VALVE_REG, J13 OUTPUTS, J14 VALVES_FRONT, J15 VALVES_BACK, J2 UART_DEBUG, J3 DEBUG, J4 EXPANSION, J5 SWD, J6 CAN, J7 USB_B_Micro, J8 BUTTONS, J9 ENGINE, Q1 IPD30N06S4L23, Q10 IPD30N06S4L23, Q11 IPD30N06S4L23, Q12 IPD30N06S4L23, Q13 IPD30N06S4L23, Q2 IPD30N06S4L23, Q3 DMP2035, Q4 IPD30N06S4L23, Q5 IPD30N06S4L23, Q6 IPD30N06S4L23, Q7 IPD30N06S4L23, Q8 IPD30N06S4L23, Q9 IPD30N06S4L23, SW1 RESET, U1 M24C64, U2 STM32F072RBTx, U3 TS1117BCW33, U4 MCP2562-E-SN, U5 USB6B1, U6 74HC4050, U7 74HC4050, U8 TSV912, Y1 MCSJK-7U-16.00

Commit message: Fixed opamp on ecu board to one with correct power range
Parts:
- U8: value TSV912 -> TS912
Changed lines of the file:
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@@
       (effects (font (size 1 1) (thickness 0.15)))
     )
-    (fp_text value TSV912 (at 0 3.5) (layer F.Fab)
+    (fp_text value TS912 (at 0 3.5) (layer F.Fab)
       (effects (font (size 1 1) (thickness 0.15)))
     )

Commit message: Reduced resistors for horn and brake buttons to switch on mosfets
Parts:
- R43, R55: value 10k -> 1k
